Commit message: ...little change

File: plutarco_description/urdf/motor.urdf.xacro (robot description, xacro)
@@ -1,5 +1,5 @@
 <?xml version="1.0"?>
-<robot xmlns:xacro="http://ros.org/wiki/xacro" name="myzharbot_motor">
-  <xacro:macro name="myzharbot_motor" params="position *joint_pose">
+<robot xmlns:xacro="http://ros.org/wiki/xacro" name="plutarco_motor">
+  <xacro:macro name="plutarco_motor" params="position *joint_pose">
     <link name="${position}_motor_link">
       <visual>

File: plutarco_description/urdf/plutarco.urdf.xacro (robot description, xacro)
@@ -1,11 +1,11 @@
 <?xml version="1.0"?>
-<robot name="myzharbot" xmlns:xacro="http://ros.org/wiki/xacro">
+<robot name="plutarco" xmlns:xacro="http://ros.org/wiki/xacro">
   <!-- Included URDF/XACRO Files -->
-  <xacro:include filename="$(find myzharbot_description)/urdf/materials.urdf" />
-  <xacro:include filename="$(find myzharbot_description)/urdf/passive_sprocket.urdf.xacro" />
-  <xacro:include filename="$(find myzharbot_description)/urdf/active_sprocket.urdf.xacro" />
-  <xacro:include filename="$(find myzharbot_description)/urdf/motor.urdf.xacro" />
-  <xacro:include filename="$(find myzharbot_description)/urdf/sensors/zed.urdf.xacro"/>
-  <xacro:include filename="$(find myzharbot_description)/urdf/sensors/imu.urdf.xacro"/>
+  <xacro:include filename="$(find plutarco_description)/urdf/materials.urdf" />
+  <xacro:include filename="$(find plutarco_description)/urdf/passive_sprocket.urdf.xacro" />
+  <xacro:include filename="$(find plutarco_description)/urdf/active_sprocket.urdf.xacro" />
+  <xacro:include filename="$(find plutarco_description)/urdf/motor.urdf.xacro" />
+  <xacro:include filename="$(find plutarco_description)/urdf/sensors/zed.urdf.xacro"/>
+  <xacro:include filename="$(find plutarco_description)/urdf/sensors/imu.urdf.xacro"/>
   <!-- Included URDF/XACRO Files -->
   <!-- Global properties -->
@@ -107,30 +107,30 @@
   <!-- Stereolabs ZED -->
   <!-- Active Sprockets -->
-  <xacro:myzharbot_active_sprocket position="Left">
+  <xacro:plutarco_active_sprocket position="Left">
     <origin xyz="${active_sprocket_offset_x} ${active_sprocket_offset_y} ${active_sprocket_offset_z}" rpy="${-M_PI/2} 0 0" />
-  </xacro:myzharbot_active_sprocket>
-  <xacro:myzharbot_active_sprocket position="Right">
+  </xacro:plutarco_active_sprocket>
+  <xacro:plutarco_active_sprocket position="Right">
     <origin xyz="${active_sprocket_offset_x} ${-active_sprocket_offset_y} ${active_sprocket_offset_z}" rpy="${-M_PI/2} 0 0" />
-  </xacro:myzharbot_active_sprocket>
-  <xacro:myzharbot_motor position="Left">
+  </xacro:plutarco_active_sprocket>
+  <xacro:plutarco_motor position="Left">
     <origin xyz="${active_sprocket_offset_x} ${active_sprocket_offset_y-0.07} ${active_sprocket_offset_z}" rpy="${-M_PI/2} 0 0" />
-  </xacro:myzharbot_motor>
-  <xacro:myzharbot_motor position="Right">
+  </xacro:plutarco_motor>
+  <xacro:plutarco_motor position="Right">
     <origin xyz="${active_sprocket_offset_x} ${-(active_sprocket_offset_y-0.07)} ${active_sprocket_offset_z}" rpy="${-M_PI/2} 0 0" />
-  </xacro:myzharbot_motor>
+  </xacro:plutarco_motor>
   <!-- Active Sprockets -->
   <!-- Passive Sprockets -->
-  <xacro:myzharbot_passive_sprocket sprocket_suffix="bfl" position="Left">
+  <xacro:plutarco_passive_sprocket sprocket_suffix="bfl" position="Left">
     <origin xyz="${passive_sprocket_offset_x} ${passive_sprocket_offset_y} ${passive_sprocket_offset_z}" rpy="${-M_PI/2} 0 0" />
-  </xacro:myzharbot_passive_sprocket>
-  <xacro:myzharbot_passive_sprocket sprocket_suffix="brl" position="Left">
+  </xacro:plutarco_passive_sprocket>
+  <xacro:plutarco_passive_sprocket sprocket_suffix="brl" position="Left">
     <origin xyz="${-passive_sprocket_offset_x} ${passive_sprocket_offset_y} ${passive_sprocket_offset_z}" rpy="${-M_PI/2} 0 0" />
-  </xacro:myzharbot_passive_sprocket>
-  <xacro:myzharbot_passive_sprocket sprocket_suffix="bfr" position="Right">
+  </xacro:plutarco_passive_sprocket>
+  <xacro:plutarco_passive_sprocket sprocket_suffix="bfr" position="Right">
     <origin xyz="${passive_sprocket_offset_x} ${-passive_sprocket_offset_y} ${passive_sprocket_offset_z}" rpy="${-M_PI/2} 0 0" />
-  </xacro:myzharbot_passive_sprocket>
-  <xacro:myzharbot_passive_sprocket sprocket_suffix="brr" position="Right">
+  </xacro:plutarco_passive_sprocket>
+  <xacro:plutarco_passive_sprocket sprocket_suffix="brr" position="Right">
     <origin xyz="${-passive_sprocket_offset_x} ${-passive_sprocket_offset_y} ${passive_sprocket_offset_z}" rpy="${-M_PI/2} 0 0" />
-  </xacro:myzharbot_passive_sprocket>
+  </xacro:plutarco_passive_sprocket>
   <!-- Passive Sprockets -->
 </robot>

File: plutarco_description/urdf/sensors/asus_xtion_pro.urdf.xacro (robot description, xacro)
@@ -30,5 +30,5 @@
         <origin xyz="-0.01 0 0" rpy="${-M_PI/2} -${M_PI} ${-M_PI/2}"/>
         <geometry>
-          <mesh filename="package://ros_myzharbot_robot/meshes/sensors/asus_xtion_pro_live.dae" scale="${M_SCALE} ${M_SCALE} ${M_SCALE}"/>
+          <mesh filename="package://ros_plutarco_robot/meshes/sensors/asus_xtion_pro_live.dae" scale="${M_SCALE} ${M_SCALE} ${M_SCALE}"/>
         </geometry>
         <material name="DarkGrey" />

File: plutarco_description/urdf/sensors/zed.urdf.xacro (robot description, xacro)
@@ -30,5 +30,5 @@
         <origin xyz="-0.01 0 0" rpy="${-M_PI/2} -${M_PI} ${-M_PI/2}"/>
         <geometry>
-          <mesh filename="package://myzharbot_description/meshes/sensors/stereolabs_zed.STL" scale="${M_SCALE} ${M_SCALE} ${M_SCALE}"/>
+          <mesh filename="package://plutarco_description/meshes/sensors/stereolabs_zed.STL" scale="${M_SCALE} ${M_SCALE} ${M_SCALE}"/>
         </geometry>
         <material name="DarkGrey" />
