Commit message: changed some file name and disabled PID on current.

File: plutarco_description/urdf/plutarco.urdf (robot description, URDF)
Before this commit: robot example, 3 links, 2 joints
Links:
- link left_wheel: geometry collision cylinder length=0.02 radius=0.10; visual cylinder length=0.02 radius=0.10
- link right_wheel: geometry collision cylinder length=0.02 radius=0.05; visual cylinder length=0.02 radius=0.10

Commit message: Configuration improving.

File: plutarco_description/urdf/plutarco.urdf (robot description, URDF)
Before this commit: robot plutarco, 3 links, 2 joints
Links:
- link base_link: geometry visual box size=0.89 0.35 0.14

Commit message: xacro update

File: plutarco_description/urdf/plutarco.urdf (robot description, URDF)
Before this commit: robot plutarco, 3 links, 2 joints
Links:
- link base_link: geometry visual box size=0.89 0.35 0.16
- link left_wheel: geometry collision cylinder length=0.02 radius=0.10; visual cylinder length=0.09 radius=0.105
- link right_wheel: geometry collision cylinder length=0.02 radius=0.05; visual cylinder length=0.09 radius=0.105
Joints:
- joint left_joint: origin xyz=0 0.1 0.05 rpy=1.57075 0.0 0.0 -> xyz=0 0.22 0.05 rpy=1.57075 0.0 0.0
- joint right_joint: origin xyz=0 -0.1 0.05 rpy=1.57075 0.0 0.0 -> xyz=0 -0.22 0.05 rpy=1.57075 0.0 0.0

File: plutarco_description/urdf/plutarco.urdf.xacro (robot description, xacro)
@@ -4,8 +4,8 @@
   <xacro:include filename="$(find plutarco_description)/urdf/materials.urdf" />
   <xacro:include filename="$(find plutarco_description)/urdf/motor.urdf.xacro" />
-  <xacro:include filename="$(find plutarco_description)/urdf/omniwheel.urdf.xacro" />
-  <xacro:include filename="$(find plutarco_description)/urdf/wheel.urdf.xacro" />
-  <xacro:include filename="$(find plutarco_description)/urdf/asus_xtion_pro.urdf.xacro"/>
-  <xacro:include filename="$(find plutarco_description)/urdf/imu.urdf.xacro"/>
+  <!-- <xacro:include filename="$(find plutarco_description)/urdf/omniwheel.urdf.xacro" /> -->
+  <!-- <xacro:include filename="$(find plutarco_description)/urdf/wheel.urdf.xacro" /> -->
+  <!-- <xacro:include filename="$(find plutarco_description)/urdf/asus_xtion_pro.urdf.xacro"/> -->
+  <!-- <xacro:include filename="$(find plutarco_description)/urdf/imu.urdf.xacro"/> -->
   <!-- Included URDF/XACRO Files -->
   <!-- Global properties -->
@@ -21,5 +21,5 @@
   <!-- Wheels params -->
   <!-- Asus Xtion params -->
-  <xacro:property name="camera_axis" value="fixed"/>
+  <!--<xacro:property name="camera_axis" value="fixed"/>
   <xacro:property name="cam_px" value="-0.005" />
   <xacro:property name="cam_py" value="0.0" />
@@ -27,5 +27,5 @@
   <xacro:property name="cam_or" value="0" />
   <xacro:property name="cam_op" value="0" />
-  <xacro:property name="cam_oy" value="0" />
+  <xacro:property name="cam_oy" value="0" />  -->
   <!-- Asus Xtion params -->
   <xacro:macro name="plutarco_robot">
@@ -62,5 +62,5 @@
   <!-- base_link -->
   <!-- Body chassis -->
-  <link name="wall_body_Link">
+<!--   <link name="wall_body_Link">
     <inertial>
       <origin xyz="-0.090836 0 0.084998" rpy="0 0 0" />
@@ -88,5 +88,6 @@
     <axis xyz="0 0 0" />
   </joint>
-  <link name="column_body_Link">
+-->
+<!--  <link name="column_body_Link">
     <inertial>
       <origin xyz="-0.11 0.00119 0.05782" rpy="0 0 0" />
@@ -111,5 +112,6 @@
     <axis xyz="0 0 0" />
   </joint>
-  <link name="battery_Link">
+-->
+<!--  <link name="battery_Link">
     <inertial>
       <origin xyz="0 0 0.018" rpy="0 0 0" />
@@ -134,5 +136,6 @@
     <axis xyz="0 0 0" />
   </joint>
-  <link name="electronics_Link">
+-->
+<!--  <link name="electronics_Link">
     <inertial>
       <origin xyz="-0.036996 0.030509 0.06534" rpy="0 0 0" />
@@ -157,5 +160,6 @@
     <axis xyz="0 0 0" />
   </joint>
-  <link name="jetson_board_Link">
+-->
+<!--  <link name="jetson_board_Link">
     <inertial>
       <origin xyz="-0.014974 0.000698 0.0046671" rpy="0 0 0" />
@@ -180,35 +184,41 @@
     <axis xyz="0 0 0" />
   </joint>
+-->
   <!-- IMU -->
+  <!--
   <xacro:imu name="base_imu" parent="base_link">
-    <!--<origin xyz="-0.06 0 0.11" rpy="0 0 0" />-->
     <origin xyz="-0.0617 -0.0008 0.1043376" rpy="0 0 0" />
   </xacro:imu>
+-->
   <!-- IMU -->
   <!-- Motors -->
-  <xacro:motor position="left" parent="column_body_Link">
+  <xacro:motor position="left" parent="base_link">
     <origin xyz="0 0.087616 0.0365" rpy="0 0 0" />
   </xacro:motor>
-  <xacro:motor position="right" parent="column_body_Link">
+  <xacro:motor position="right" parent="base_link">
     <origin xyz="0 -0.087616 0.0365" rpy="0 0 ${M_PI}" />
   </xacro:motor>
   <!-- Motors -->
   <!-- Omniwheel -->
+  <!--
   <xacro:omniwheel parent="base_link">
     <origin xyz="-0.20895 0 0.021838" rpy="0 0 ${M_PI}" />
   </xacro:omniwheel>
+-->
   <!-- Omniwheel -->
   <!-- Asus Xtion Pro Live -->
+  <!--
   <xacro:sensor_asus_xtion_pro parent="base_link" type="${camera_axis}">
     <origin xyz="${cam_px} ${cam_py} ${cam_pz}"  rpy="${cam_or} ${cam_op} ${cam_oy}" />
   </xacro:sensor_asus_xtion_pro>
+-->
   <!-- Asus Xtion Pro Live -->
   <!-- Wheels -->
-  <xacro:banebots_wheel position="Left" reflect="-1">
+  <xacro:plutarco_traction_gear position="Left" reflect="-1">
     <origin xyz="${wheel_offset_x} ${-wheel_offset_y} ${wheel_offset_z}" rpy="${M_PI/2} 0 0" />
-  </xacro:banebots_wheel>
-  <xacro:banebots_wheel position="Right" reflect="1">
+  </xacro:plutarco_traction_gear>
+  <xacro:plutarco_traction_gear position="Right" reflect="1">
     <origin xyz="${wheel_offset_x} ${wheel_offset_y} ${wheel_offset_z}" rpy="${-M_PI/2} 0 0" />
-  </xacro:banebots_wheel>
+  </xacro:plutarco_traction_gear>
   <!-- Wheels -->
   </xacro:macro>

Commit message: Initial plutarco_statup.launch file

File: plutarco_description/urdf/plutarco.urdf (robot description, URDF)
Before this commit: robot plutarco, 3 links, 2 joints
Links:
- added link camera_link; collision box size=0.01 0.14 0.02; visual box size=0.01 0.14 0.02
- added link imu_link; collision box size=0.02 0.03 0.005; visual box size=0.02 0.03 0.005
- added link rplidar_link; visual cylinder length=0.06 radius=0.035
- added link ydlidar_link; visual cylinder length=0.06 radius=0.035
- link base_link: geometry visual box size=0.55 0.89 0.24
- link left_wheel: geometry collision cylinder length=0.06 radius=0.1; visual cylinder length=0.06 radius=0.1
- link right_wheel: geometry collision cylinder length=0.06 radius=0.1; visual cylinder length=0.06 radius=0.1
Joints:
- added joint base_link_to_base_laser_rp: type fixed, parent base_link, child rplidar_link, origin xyz=-0.07 0 0.35 rpy=0 0 -1.5708
- added joint base_link_to_base_laser_yd: type fixed, parent base_link, child ydlidar_link, origin xyz=-0.07 0.12 0.38 rpy=0 0 -1.5708
- added joint camera_joint: type fixed, parent base_link, child camera_link, origin xyz=0.045 0.00 0.094 rpy=0.0 0.0 0.0
- added joint imu_joint: type fixed, parent base_link, child imu_link, origin xyz=-0.025 0.05 0.11 rpy=0.0 0.0 0.0
- joint left_joint: origin xyz=0 0.22 0.05 rpy=1.57075 0.0 0.0 -> xyz=0 0.07 0.0365125 rpy=1.57075 0.0 0.0
- joint right_joint: origin xyz=0 -0.22 0.05 rpy=1.57075 0.0 0.0 -> xyz=0 -0.07 0.0365125 rpy=1.57075 0.0 0.0

Commit message: little URDF and startup launch file improve.

File: plutarco_description/urdf/plutarco.urdf (robot description, URDF)
Before this commit: robot plutarco, 7 links, 6 joints
Links:
- removed link camera_link
- added link ZED_center; collision box size=0.01 0.14 0.02; visual box size=0.01 0.14 0.02
- link base_link: geometry visual box size=0.89 0.55 0.24
Joints:
- joint camera_joint: child camera_link -> ZED_center
- joint left_joint: origin xyz=0 0.07 0.0365125 rpy=1.57075 0.0 0.0 -> xyz=0 0.28 0.0365125 rpy=1.57075 0.0 0.0
- joint right_joint: origin xyz=0 -0.07 0.0365125 rpy=1.57075 0.0 0.0 -> xyz=0 -0.28 0.0365125 rpy=1.57075 0.0 0.0

Commit message: First real URDF PlutarcoÃ's model

File: plutarco_description/urdf/plutarco.urdf (robot description, URDF)
Before this commit: robot plutarco, 7 links, 6 joints
Links:
- removed link ZED_center
- added link body_main; visual mesh filename=package://plutarco_description/urdf/models/Body.stl scale=0.001 0.001 0.001
- link base_link: geometry visual cylinder length=0.001 radius=0.03
Joints:
- removed joint camera_joint
- added joint body_main_joint: type fixed, parent base_link, child body_main, origin xyz=0.0 0.00 -0.14 rpy=1.5708 0.0 0.0
- joint base_link_to_base_laser_rp: origin xyz=-0.07 0 0.35 rpy=0 0 -1.5708 -> xyz=-0.07 0 0.35 rpy=0 0 0
- joint left_joint: origin xyz=0 0.28 0.0365125 rpy=1.57075 0.0 0.0 -> xyz=0 0.28 -0.17 rpy=1.57075 0.0 0.0
- joint right_joint: origin xyz=0 -0.28 0.0365125 rpy=1.57075 0.0 0.0 -> xyz=0 -0.28 -0.17 rpy=1.57075 0.0 0.0

Commit message: Update URDF model

File: plutarco_description/urdf/plutarco.urdf (robot description, URDF)
Before this commit: robot plutarco, 7 links, 6 joints
Links:
- removed link ydlidar_link
- added link plutarco_head; visual mesh filename=package://plutarco_description/urdf/models/Plutarco_Head.stl scale=0.001 0.001 0.001
Joints:
- removed joint base_link_to_base_laser_yd
- added joint plutarco_head_joint: type fixed, parent body_main, child plutarco_head, origin xyz=0.0 0.23 -0.05 rpy=0.0 0.0 0.0
- joint base_link_to_base_laser_rp: origin xyz=-0.07 0 0.35 rpy=0 0 0 -> xyz=-0.10 0.00 0.32 rpy=0 0 3.14159
- joint body_main_joint: origin xyz=0.0 0.00 -0.14 rpy=1.5708 0.0 0.0 -> xyz=0.0 0.0 0.0 rpy=1.5708 0.0 1.5708
- joint imu_joint: origin xyz=-0.025 0.05 0.11 rpy=0.0 0.0 0.0 -> xyz=0.0 0.0 0.0 rpy=0.0 0.0 0.0

Commit message: general improving

File: plutarco_description/urdf/plutarco.urdf (robot description, URDF)
Before this commit: robot plutarco, 7 links, 6 joints
Links:
- link body_main: geometry visual mesh filename=package://robot_description/urdf/models/Body.stl scale=0.001 0.001 0.001
- link plutarco_head: geometry visual mesh filename=package://robot_description/urdf/models/Plutarco_Head.stl scale=0.001 0.001 0.001
